File: hardware/e24-receiver-board/production/e24-receiver-board.kicad_pcb (KiCad board)
At the start: 2 copper layers, 70 x 70 mm, 307 parts, among them J1 505070-2422, J10 SPEAKER-, J11 GND1, J12 TRACK_RIGHT, J13 MOTOR+, J14 LAMP_REAR, J15 CAP+, J16 U+, J17 AUX3, J18 AUX10, J19 AUX12, J2 TRACK_LEFT, J20 SPEAKER+, J21 GND2, J3 MOTOR-, J4 LAMP_FRONT, J5 VCC, J6 AUX1, J7 AUX2, J8 AUX4, J9 AUX11

Commit message: fix: update connector part number
Parts:
- J1 (x4): value 505070-2422 -> 5052742412
