File: hardware/pico2-test-mule/pico2-test-mule.kicad_pcb (KiCad board)
At the start: 2 copper layers, 52.5 x 42 mm, 70 parts, among them J1 SPEAKER, J2 POWER, J3 AUX, J4 MOTOR, J5 VCC, Q1 DMN2991UDA-7B, Q10 DMN2991UDA-7B, Q11 DMN2991UDA-7B, Q12 DMN2991UDA-7B, Q13 DMN2991UDA-7B, Q2 SS8050, Q3 SS8050, Q4 DMN2991UDA-7B, Q5 SS8050, Q6 SS8050, Q7 NST847BPDP6T5G, Q8 SS8050, Q9 NST847BPDP6T5G, U1 NCS2220AMUT1G, U2 AP63203WU, U3 PICO, U4 MAX98357AEWL+T, U5 MD9927

Commit message: chore: export footprints to library
Parts:
- C1, C10, C3, C7, C9: footprint Capacitor_SMD:C_0402_1005Metric -> pico2-test-mule:C_0402_1005Metric
- C2, C4: footprint Capacitor_SMD:C_0603_1608Metric -> pico2-test-mule:C_0603_1608Metric
- C5, C8: footprint Capacitor_SMD:C_1206_3216Metric -> pico2-test-mule:C_1206_3216Metric
- C6: footprint Capacitor_SMD:C_0805_2012Metric -> pico2-test-mule:C_0805_2012Metric
- D10, D11, D12, D14, D15, D16, D17, D19, D3, D4, D5, D6, D9: footprint LED_SMD:LED_0603_1608Metric -> pico2-test-mule:LED_0603_1608Metric
- J1: footprint Connector_PinHeader_2.54mm:PinHeader_1x06_P2.54mm_Vertical -> pico2-test-mule:PinHeader_1x06_P2.54mm_Vertical
- J2: footprint Connector_PinHeader_2.54mm:PinHeader_1x04_P2.54mm_Vertical -> pico2-test-mule:PinHeader_1x04_P2.54mm_Vertical
- J3: footprint Connector_PinHeader_2.54mm:PinHeader_1x05_P2.54mm_Vertical -> pico2-test-mule:PinHeader_1x05_P2.54mm_Vertical
- J4, J5: footprint Connector_PinHeader_2.54mm:PinHeader_1x02_P2.54mm_Vertical -> pico2-test-mule:PinHeader_1x02_P2.54mm_Vertical
- Q2, Q3, Q5, Q6, Q8: footprint Package_TO_SOT_SMD:SOT-23 -> pico2-test-mule:SOT-23
- Q7, Q9: footprint Package_TO_SOT_SMD:SOT-963 -> pico2-test-mule:SOT-963
- R1, R10, R11, R12, R13, R14, R2, R3, R4, R5, R6, R7, R8, R9: footprint Resistor_SMD:R_0402_1005Metric -> pico2-test-mule:R_0402_1005Metric
- RN1, RN2, RN3: footprint Resistor_SMD:R_Array_Concave_4x0402 -> pico2-test-mule:R_Array_Concave_4x0402
- U3: footprint Module:RaspberryPi_Pico_Common_THT -> pico2-test-mule:RaspberryPi_Pico_Common_THT
Changed lines of the file:
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@@
 		)
 	)
-	(footprint "Package_TO_SOT_SMD:SOT-963"
+	(footprint "pico2-test-mule:SOT-963"
 		(layer "F.Cu")
 		(at 117.3 66.25 90)
@@
 		)
 	)
-	(footprint "Resistor_SMD:R_0402_1005Metric"
+	(footprint "pico2-test-mule:R_0402_1005Metric"
 		(layer "F.Cu")
 		(at 117.3 68.25 90)
@@
 		)
 	)
-	(footprint "Resistor_SMD:R_0402_1005Metric"
+	(footprint "pico2-test-mule:R_0402_1005Metric"
 		(layer "F.Cu")
 		(at 116.25 68.25 90)
@@
 		)
 	)
-	(footprint "Resistor_SMD:R_Array_Concave_4x0402"
+	(footprint "pico2-test-mule:R_Array_Concave_4x0402"
 		(layer "F.Cu")
 		(at 104.2 75.2725 -90)
@@
 		)
 	)
-	(footprint "LED_SMD:LED_0603_1608Metric"
+	(footprint "pico2-test-mule:LED_0603_1608Metric"
 		(layer "F.Cu")
 		(at 105.025 78.185 90)
@@
 		)
 	)
-	(footprint "LED_SMD:LED_0603_1608Metric"
+	(footprint "pico2-test-mule:LED_0603_1608Metric"
 		(layer "F.Cu")
 		(at 112 78.185 90)
@@
 		)
 	)
-	(footprint "Capacitor_SMD:C_0402_1005Metric"
+	(footprint "pico2-test-mule:C_0402_1005Metric"
 		(layer "F.Cu")
 		(at 99.15 66.1 180)
@@
 		)
 	)
-	(footprint "Connector_PinHeader_2.54mm:PinHeader_1x02_P2.54mm_Vertical"
+	(footprint "pico2-test-mule:PinHeader_1x02_P2.54mm_Vertical"
 		(layer "F.Cu")
 		(at 98.275 61.4 90)
@@
 		)
 	)
-	(footprint "LED_SMD:LED_0603_1608Metric"
+	(footprint "pico2-test-mule:LED_0603_1608Metric"
 		(layer "F.Cu")
 		(at 102.7 78.185 90)
@@
 		)
 	)
-	(footprint "Package_TO_SOT_SMD:SOT-23"
+	(footprint "pico2-test-mule:SOT-23"
 		(layer "F.Cu")
 		(at 116.6 74.3725 -90)
@@
 		)
 	)
-	(footprint "Capacitor_SMD:C_0402_1005Metric"
+	(footprint "pico2-test-mule:C_0402_1005Metric"
 		(layer "F.Cu")
 		(at 109 67.05)
@@
 		)
 	)
-	(footprint "Resistor_SMD:R_Array_Concave_4x0402"
+	(footprint "pico2-test-mule:R_Array_Concave_4x0402"
 		(layer "F.Cu")
 		(at 94.8 75.285 -90)
@@
 		)
 	)
-	(footprint "Connector_PinHeader_2.54mm:PinHeader_1x04_P2.54mm_Vertical"
+	(footprint "pico2-test-mule:PinHeader_1x04_P2.54mm_Vertical"
 		(layer "F.Cu")
 		(at 125.11 77.935 90)
@@
 		)
 	)
-	(footprint "Resistor_SMD:R_0402_1005Metric"
+	(footprint "pico2-test-mule:R_0402_1005Metric"
 		(layer "F.Cu")
 		(at 120.45 68.25 -90)
@@
 		)
 	)
-	(footprint "Module:RaspberryPi_Pico_Common_THT"
+	(footprint "pico2-test-mule:RaspberryPi_Pico_Common_THT"
 		(locked yes)
 		(layer "F.Cu")
@@
 		)
 	)
-	(footprint "Resistor_SMD:R_Array_Concave_4x0402"
+	(footprint "pico2-test-mule:R_Array_Concave_4x0402"
 		(layer "F.Cu")
 		(at 113.6 75.2725 -90)
@@
 		)
 	)
-	(footprint "Resistor_SMD:R_0402_1005Metric"
+	(footprint "pico2-test-mule:R_0402_1005Metric"
 		(layer "F.Cu")
 		(at 109 70.85)
@@
 		)
 	)
-	(footprint "Connector_PinHeader_2.54mm:PinHeader_1x06_P2.54mm_Vertical"
+	(footprint "pico2-test-mule:PinHeader_1x06_P2.54mm_Vertical"
 		(layer "F.Cu")
 		(at 90.3 64.47)
@@
 		)
 	)
-	(footprint "Capacitor_SMD:C_1206_3216Metric"
+	(footprint "pico2-test-mule:C_1206_3216Metric"
 		(layer "F.Cu")
 		(at 106.49 68.95 -90)
@@
 		)
 	)
-	(footprint "Resistor_SMD:R_0402_1005Metric"
+	(footprint "pico2-test-mule:R_0402_1005Metric"
 		(layer "F.Cu")
 		(at 119.4 75.285 -90)
@@
 		)
 	)
-	(footprint "LED_SMD:LED_0603_1608Metric"
+	(footprint "pico2-test-mule:LED_0603_1608Metric"
 		(layer "F.Cu")
 		(at 107.35 78.185 90)
@@
 		)
 	)
-	(footprint "Resistor_SMD:R_0402_1005Metric"
+	(footprint "pico2-test-mule:R_0402_1005Metric"
 		(layer "F.Cu")
 		(at 96.71 64.05 180)
@@
 		)
 	)
-	(footprint "Capacitor_SMD:C_0805_2012Metric"
+	(footprint "pico2-test-mule:C_0805_2012Metric"
 		(layer "F.Cu")
 		(at 119.82 70.35)
@@
 		)
 	)
-	(footprint "LED_SMD:LED_0603_1608Metric"
+	(footprint "pico2-test-mule:LED_0603_1608Metric"
 		(layer "F.Cu")
 		(at 121.3 78.185 90)
@@
 		)
 	)
-	(footprint "Capacitor_SMD:C_0603_1608Metric"
+	(footprint "pico2-test-mule:C_0603_1608Metric"
 		(layer "F.Cu")
 		(at 109.95 63.955 90)
@@
 		)
 	)
-	(footprint "Package_TO_SOT_SMD:SOT-963"
+	(footprint "pico2-test-mule:SOT-963"
 		(layer "F.Cu")
 		(at 117.3 70.3 -90)
@@
 		)
 	)
-	(footprint "Resistor_SMD:R_0402_1005Metric"
+	(footprint "pico2-test-mule:R_0402_1005Metric"
 		(layer "F.Cu")
 		(at 109 68)
@@
 		)
 	)
-	(footprint "LED_SMD:LED_0603_1608Metric"
+	(footprint "pico2-test-mule:LED_0603_1608Metric"
 		(layer "F.Cu")
 		(at 98.05 78.185 90)
@@
 		)
 	)
-	(footprint "Resistor_SMD:R_0402_1005Metric"
+	(footprint "pico2-test-mule:R_0402_1005Metric"
 		(layer "F.Cu")
 		(at 109 68.95)
@@
 		)
 	)
-	(footprint "Connector_PinHeader_2.54mm:PinHeader_1x02_P2.54mm_Vertical"
+	(footprint "pico2-test-mule:PinHeader_1x02_P2.54mm_Vertical"
 		(layer "F.Cu")
 		(at 121.775 63.6 90)
@@
 		)
 	)
-	(footprint "Resistor_SMD:R_0402_1005Metric"
+	(footprint "pico2-test-mule:R_0402_1005Metric"
 		(layer "F.Cu")
 		(at 96.71 66 180)
@@
 		)
 	)
-	(footprint "Package_TO_SOT_SMD:SOT-23"
+	(footprint "pico2-test-mule:SOT-23"
 		(layer "F.Cu")
 		(at 101.2 74.7725 -90)
@@
 		)
 	)
-	(footprint "Package_TO_SOT_SMD:SOT-23"
+	(footprint "pico2-test-mule:SOT-23"
 		(layer "F.Cu")
 		(at 107.2 74.435 -90)
@@
 		)
 	)
-	(footprint "LED_SMD:LED_0603_1608Metric"
+	(footprint "pico2-test-mule:LED_0603_1608Metric"
 		(layer "F.Cu")
 		(at 95.725 78.185 90)
@@
 		)
 	)
-	(footprint "Capacitor_SMD:C_1206_3216Metric"
+	(footprint "pico2-test-mule:C_1206_3216Metric"
 		(layer "F.Cu")
 		(at 104.19 68.95 -90)
@@
 		)
 	)
-	(footprint "LED_SMD:LED_0603_1608Metric"
+	(footprint "pico2-test-mule:LED_0603_1608Metric"
 		(layer "F.Cu")
 		(at 100.375 78.185 90)
@@
 		)
 	)
-	(footprint "LED_SMD:LED_0603_1608Metric"
+	(footprint "pico2-test-mule:LED_0603_1608Metric"
 		(layer "F.Cu")
 		(at 116.65 78.185 90)
@@
 		)
 	)
-	(footprint "Capacitor_SMD:C_0402_1005Metric"
+	(footprint "pico2-test-mule:C_0402_1005Metric"
 		(layer "F.Cu")
 		(at 101.38 70.55)
@@
 		)
 	)
-	(footprint "Resistor_SMD:R_0402_1005Metric"
+	(footprint "pico2-test-mule:R_0402_1005Metric"
 		(layer "F.Cu")
 		(at 118.35 68.2475 90)
@@
 		)
 	)
-	(footprint "Resistor_SMD:R_0402_1005Metric"
+	(footprint "pico2-test-mule:R_0402_1005Metric"
 		(layer "F.Cu")
 		(at 109 69.9)
@@
 		)
 	)
-	(footprint "Resistor_SMD:R_0402_1005Metric"
+	(footprint "pico2-test-mule:R_0402_1005Metric"
 		(layer "F.Cu")
 		(at 96.71 65)
@@
 		)
 	)
-	(footprint "Capacitor_SMD:C_0402_1005Metric"
+	(footprint "pico2-test-mule:C_0402_1005Metric"
 		(layer "F.Cu")
 		(at 105.8 62.105 180)
@@
 		)
 	)
-	(footprint "Capacitor_SMD:C_0603_1608Metric"
+	(footprint "pico2-test-mule:C_0603_1608Metric"
 		(layer "F.Cu")
 		(at 101.9 64.25 90)
@@
 		)
 	)
-	(footprint "LED_SMD:LED_0603_1608Metric"
+	(footprint "pico2-test-mule:LED_0603_1608Metric"
 		(layer "F.Cu")
 		(at 118.975 78.185 90)
@@
 		)
 	)
-	(footprint "Resistor_SMD:R_0402_1005Metric"
+	(footprint "pico2-test-mule:R_0402_1005Metric"
 		(layer "F.Cu")
 		(at 96.71 66.95 180)
@@
 		)
 	)
-	(footprint "Package_TO_SOT_SMD:SOT-23"
+	(footprint "pico2-test-mule:SOT-23"
 		(layer "F.Cu")
 		(at 110.6 74.435 -90)
@@
 		)
 	)
-	(footprint "LED_SMD:LED_0603_1608Metric"
+	(footprint "pico2-test-mule:LED_0603_1608Metric"
 		(layer "F.Cu")
 		(at 93.4 78.185 90)
@@
 		)
 	)
-	(footprint "Capacitor_SMD:C_0402_1005Metric"
+	(footprint "pico2-test-mule:C_0402_1005Metric"
 		(layer "F.Cu")
 		(at 101.38 69.6)
@@
 		)
 	)
-	(footprint "LED_SMD:LED_0603_1608Metric"
+	(footprint "pico2-test-mule:LED_0603_1608Metric"
 		(layer "F.Cu")
 		(at 109.675 78.185 90)
@@
 		)
 	)
-	(footprint "Package_TO_SOT_SMD:SOT-23"
+	(footprint "pico2-test-mule:SOT-23"
 		(layer "F.Cu")
 		(at 97.8 74.7725 -90)
@@
 		)
 	)
-	(footprint "Resistor_SMD:R_0402_1005Metric"
+	(footprint "pico2-test-mule:R_0402_1005Metric"
 		(layer "F.Cu")
 		(at 119.4 68.25 -90)
@@
 		)
 	)
-	(footprint "Connector_PinHeader_2.54mm:PinHeader_1x05_P2.54mm_Vertical"
+	(footprint "pico2-test-mule:PinHeader_1x05_P2.54mm_Vertical"
 		(layer "F.Cu")
 		(at 122.56 74.05 90)
@@
 		)
 	)
-	(footprint "LED_SMD:LED_0603_1608Metric"
+	(footprint "pico2-test-mule:LED_0603_1608Metric"
 		(layer "F.Cu")
 		(at 114.325 78.185 90)

Commit message: fix: reduce DCC_TTL gate voltage
fix: tweak DCC_TTL debounce cap value
Parts:
- C6: value 10nF -> 470pF
- R6: value 6.8K -> 2.2K
Changed lines of the file:
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@@
 			)
 		)
-		(property "Value" "6.8K"
+		(property "Value" "2.2K"
 			(at 0 1.17 90)
 			(layer "F.Fab")
@@
 			)
 		)
-		(property "LCSC" "C25944"
+		(property "LCSC" "C25879"
 			(at 0 0 90)
 			(unlocked yes)
@@
 			)
 		)
-		(property "Value" "10nF"
+		(property "Value" "470pF"
 			(at 0 1.68 0)
 			(layer "F.Fab")
@@
 			)
 		)
-		(property "LCSC" "C1710"
+		(property "LCSC" "C1743"
 			(at 0 0 0)
 			(unlocked yes)
