File: hardware/e24-receiver-board/e24-receiver-board.kicad_pcb (KiCad board)
At the start: 2 copper layers, 24 x 8.6 mm, 21 parts, among them J1 505070-2422, J10 SPEAKER-, J11 GND1, J12 TRACK_RIGHT, J13 MOTOR+, J14 LAMP_REAR, J15 CAP+, J16 U+, J17 AUX3, J18 AUX10, J19 AUX12, J2 TRACK_LEFT, J20 SPEAKER+, J21 GND2, J3 MOTOR-, J4 LAMP_FRONT, J5 VCC, J6 AUX1, J7 AUX2, J8 AUX4, J9 AUX11

Commit message: fix: update connector part number
Parts:
- J1: value 505070-2422 -> 5052742412
Changed lines of the file:
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@@
 			)
 		)
-		(property "Value" "505070-2422"
+		(property "Value" "5052742412"
 			(at 0 -4.91 90)
 			(layer "B.Fab")
@@
 			)
 		)
-		(property "Datasheet" "https://componentsearchengine.com/Datasheets/1/505070-2422.pdf"
+		(property "Datasheet" "https://componentsearchengine.com/Datasheets/1/505274-2412.pdf"
 			(at 0 0 90)
 			(layer "B.Fab")
@@
 			)
 		)
-		(property "Manufacturer_Name" "Molex"
+		(property "LCSC" "C3649712"
 			(at 0 0 90)
 			(unlocked yes)
 			(layer "B.Fab")
-			(hide yes)
-			(effects
-				(font
-					(size 1 1)
-					(thickness 0.15)
-				)
-				(justify mirror)
-			)
-		)
-		(property "Manufacturer_Part_Number" "505070-2422"
-			(at 0 0 90)
-			(unlocked yes)
-			(layer "B.Fab")
-			(hide yes)
-			(effects
-				(font
-					(size 1 1)
-					(thickness 0.15)
-				)
-				(justify mirror)
-			)
-		)
-		(property "LCSC" "C724143"
-			(at 0 0 90)
-			(unlocked yes)
-			(layer "B.Fab")
-			(hide yes)
-			(effects
-				(font
-					(size 1 1)
-					(thickness 0.15)
-				)
-				(justify mirror)
-			)
-		)
-		(property "Description_1" ""
-			(at 0 0 270)
-			(unlocked yes)
-			(layer "B.Fab")
-			(hide yes)
-			(effects
-				(font
-					(size 1 1)
-					(thickness 0.15)
-				)
-				(justify mirror)
-			)
-		)
-		(property "Mouser Part Number" ""
-			(at 0 0 270)
-			(unlocked yes)
-			(layer "B.Fab")
-			(hide yes)
-			(effects
-				(font
-					(size 1 1)
-					(thickness 0.15)
-				)
-				(justify mirror)
-			)
-		)
-		(property "Mouser Price/Stock" ""
-			(at 0 0 270)
-			(unlocked yes)
-			(layer "B.Fab")
