File: hardware/rp24-usb-tester/rp24-usb-tester.kicad_pcb (KiCad board)
At the start: 2 copper layers, 50 x 25 mm, 40 parts, among them J1 SPEAKER, J2 POWER, J3 EXT_CAP, J4 505070-2422, J5 RAILS, J6 AUX, J7 MOTOR, P1 USB_C_Receptacle_USB2.0_16P, Q1 SS8050, Q2 SS8050, Q3 SS8050, Q4 SS8050, Q5 SS8050, U1 MT2492

Commit message: fix: bump resistors to make LEDs less blinding
Parts:
- RN1, RN2, RN3: value R_Pack04 -> 220R
Changed lines of the file:
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@@
 			)
 		)
-		(property "Value" "R_Pack04"
+		(property "Value" "220R"
 			(at 0 2.1 0)
 			(layer "F.Fab")
@@
 			)
 		)
-		(property "LCSC" "C48442"
+		(property "LCSC" "C326868"
 			(at 0 0 0)
 			(unlocked yes)
@@
 			)
 		)
-		(property "Value" "R_Pack04"
+		(property "Value" "220R"
 			(at 0 2.1 180)
 			(layer "F.Fab")
@@
 			)
 		)
-		(property "LCSC" "C48442"
+		(property "LCSC" "C326868"
 			(at 0 0 180)
 			(unlocked yes)
@@
 			)
 		)
-		(property "Value" "R_Pack04"
+		(property "Value" "220R"
 			(at 0 2.1 270)
 			(layer "F.Fab")
@@
 			)
 		)
-		(property "LCSC" "C48442"
+		(property "LCSC" "C326868"
 			(at 0 0 270)
 			(unlocked yes)
